File: LabReports/Lab2/David_Smith-smd.brd (EAGLE design)
At the start: 51.7 x 33 mm, 5 parts, among them J1 2.1MMJACKTHM

Commit message: Update Lab2 turnin
Changed lines of the file:
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@@
 <wire x1="0" y1="0" x2="51.74" y2="0" width="0.254" layer="20"/>
 <wire x1="51.74" y1="0" x2="51.74" y2="33.01" width="0.254" layer="20"/>
-<wire x1="51.74" y1="33.01" x2="0" y2="33.01" width="0.254" layer="20"/>
+<wire x1="51.74" y1="33.01" x2="0" y2="33.01" width="0.254" layer="21"/>
 <wire x1="0" y1="33.01" x2="0" y2="0" width="0.254" layer="20"/>
 <dimension x1="0" y1="33.01" x2="0" y2="0" x3="-5.08" y3="16.505" textsize="1.778" layer="51" unit="inch"/>
