File: LabReports/Lab2/David_Smith-th.brd (EAGLE design)
At the start: 51.7 x 33 mm, 4 parts, among them J1 2.1MMJACKTHM

Commit message: Update Lab2 turnin
Parts:
- added U$2: (no value), Lab2:UCSD_LOGO
Changed lines of the file:
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@@
 <wire x1="0" y1="0" x2="51.74" y2="0" width="0.254" layer="20"/>
 <wire x1="51.74" y1="0" x2="51.74" y2="33.01" width="0.254" layer="20"/>
-<wire x1="51.74" y1="33.01" x2="0" y2="33.01" width="0.254" layer="20"/>
+<wire x1="51.74" y1="33.01" x2="0" y2="33.01" width="0.254" layer="21"/>
 <wire x1="0" y1="33.01" x2="0" y2="0" width="0.254" layer="20"/>
 <dimension x1="0" y1="33.01" x2="0" y2="0" x3="-5.08" y3="16.505" textsize="1.778" layer="51" unit="inch"/>
@@
 <attribute name="TOL" value="" x="41.91" y="8.89" size="1.778" layer="27" display="off"/>
 </element>
+<element name="U$2" library="Lab2" package="UCSD_LOGO" value="" x="41.91" y="29.21"/>
 </elements>
 <signals>
